File: pcb/ai_ardushield_lumina.sch (EAGLE design)
At the start: 90 parts, among them J1 1X02ST, J2 1X01, J3 1X06, J4 1X08, J5 1X08, J6 1X10, SW1 SW-SPST, U1 ARDUINOUNOR3-STRAIGHT

Commit message: Updated to latest libraries.  New Gerbers.
Parts:
- removed SW1: SW-SPST, Ai_Electromechanical:SW-SPST
- added S1: SW-SPSTSMD06X06, Ai_Electromechanical:SW-SPSTSMD06X06
- C1, C10, C11, C12, C13, C14, C15, C16, C17, C18, C19, C2, C20, C21, C22, C23, C24, C25, C26, C27, C28, C29, C3, C30, C31, C32, C33, C34, C35, C36, C37, C38, C39, C4, C40, C5, C6, C7, C8, C9: value (none) -> 0.1uF; device Ai_Passives:CAP -> Ai_Passives:CAP0603
Connections:
- net GND: now also S1.A@1; no longer C38.2, SW1.A@1, SW1.A@2
- net RST: now also S1.B@1; no longer SW1.B@1, SW1.B@2
Other:
- moved on the sheet: C12, C13, C14, C15, C16, C20, C21, C22, C23, C24, C28, C29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
